File: plenum/plenum.kicad_pcb (KiCad board)
At the start: 2 copper layers, 87 parts, among them J1 Conn_02x01, J3 Conn_03x20_MountingPin, J4 Conn_02x10_Row_Letter_First, U1 PIC18F66J60-IPT, U10 NBA3N011S, U11 NBA3N011S, U12 NBA3N011S, U13 NBA3N011S, U14 NBA3N011S, U15 NBA3N011S, U16 TPS62082, U17 TPS54294, U18 LTC2983, U19 LTC2983, U3 74LVC1G02, U4 74LVC1G02, U6 NBA3N011S, U7 NBA3N011S, U8 NBA3N011S, U9 NBA3N011S

Commit message: adding notes and BMI270 IMU to plenum
Parts:
- added H1: MountingHole_Pad, MountingHole:MountingHole_3.2mm_M3_Pad, F.Cu at (-3.81, 3.81)
- added H2: MountingHole_Pad, MountingHole:MountingHole_3.2mm_M3_Pad, F.Cu at (-113.0, 3.81)
- added H3: MountingHole_Pad, MountingHole:MountingHole_3.2mm_M3_Pad, F.Cu at (-19.7, 55.9)
- added H4: MountingHole_Pad, MountingHole:MountingHole_3.2mm_M3_Pad, F.Cu at (-92.1, 55.9)
- added J5: RJ45_Wuerth_7498210220A, Connector_RJ:RJ45_Wuerth_7498210220A_Horizontal, F.Cu at (-108.5, 46.5)
- added U20: BMI270, Sensor_Motion:BMI270, F.Cu at (84.6, 109.5)
- J1: footprint Connector_PinHeader_1.27mm:PinHeader_1x02_P1.27mm_Vertical -> Connector_PinHeader_2.54mm:PinHeader_1x02_P2.54mm_Vertical
- moved J4 205.0 mm to (-14.6, 20.8)
- moved J3 179.5 mm to (-58.4, 50.8)
Connections:
- net /header/TEMP1.CH10 renamed /rtd_header/TEMP1.CH10
- net /header/TEMP1.CH11 renamed /rtd_header/TEMP1.CH11
- net /header/TEMP1.CH12 renamed /rtd_header/TEMP1.CH12
- net /header/TEMP1.CH13 renamed /rtd_header/TEMP1.CH13
- net /header/TEMP1.CH14 renamed /rtd_header/TEMP1.CH14
- net /header/TEMP1.CH15 renamed /rtd_header/TEMP1.CH15
- net /header/TEMP1.CH16 renamed /rtd_header/TEMP1.CH16
- net /header/TEMP1.CH17 renamed /rtd_header/TEMP1.CH17
- net /header/TEMP1.CH18 renamed /rtd_header/TEMP1.CH18
- net /header/TEMP1.CH19 renamed /rtd_header/TEMP1.CH19
- net /header/TEMP1.CH20 renamed /rtd_header/TEMP1.CH20
- net /header/TEMP1.CH3 renamed /rtd_header/TEMP1.CH3
- net /header/TEMP1.CH4 renamed /rtd_header/TEMP1.CH4
- net /header/TEMP1.CH5 renamed /rtd_header/TEMP1.CH5
- net /header/TEMP1.CH6 renamed /rtd_header/TEMP1.CH6
- net /header/TEMP1.CH7 renamed /rtd_header/TEMP1.CH7
- net /header/TEMP1.CH8 renamed /rtd_header/TEMP1.CH8
- net /header/TEMP1.CH9 renamed /rtd_header/TEMP1.CH9
- net /header/TEMP1.RSENSE renamed /rtd_header/TEMP1.RSENSE
- net /header/TEMP2.CH10 renamed /rtd_header/TEMP2.CH10
- net /header/TEMP2.CH11 renamed /rtd_header/TEMP2.CH11
- net /header/TEMP2.CH12 renamed /rtd_header/TEMP2.CH12
- net /header/TEMP2.CH13 renamed /rtd_header/TEMP2.CH13
- net /header/TEMP2.CH14 renamed /rtd_header/TEMP2.CH14
- net /header/TEMP2.CH15 renamed /rtd_header/TEMP2.CH15
- net /header/TEMP2.CH16 renamed /rtd_header/TEMP2.CH16
- net /header/TEMP2.CH17 renamed /rtd_header/TEMP2.CH17
- net /header/TEMP2.CH18 renamed /rtd_header/TEMP2.CH18
- net /header/TEMP2.CH19 renamed /rtd_header/TEMP2.CH19
- net /header/TEMP2.CH20 renamed /rtd_header/TEMP2.CH20
- net /header/TEMP2.CH3 renamed /rtd_header/TEMP2.CH3
- net /header/TEMP2.CH4 renamed /rtd_header/TEMP2.CH4
- net /header/TEMP2.CH5 renamed /rtd_header/TEMP2.CH5
- net /header/TEMP2.CH6 renamed /rtd_header/TEMP2.CH6
- net /header/TEMP2.CH7 renamed /rtd_header/TEMP2.CH7
- net /header/TEMP2.CH8 renamed /rtd_header/TEMP2.CH8
- net /header/TEMP2.CH9 renamed /rtd_header/TEMP2.CH9
- net /header/TEMP2.RSENSE renamed /rtd_header/TEMP2.RSENSE
- net /houskeeping/LDO1 renamed /rtd/LDO1
- net /houskeeping/LDO2 renamed /rtd/LDO2
- net /houskeeping/TEMP1.CH10 renamed /rtd/TEMP1.CH10
- net /houskeeping/TEMP1.CH11 renamed /rtd/TEMP1.CH11
- net /houskeeping/TEMP1.CH12 renamed /rtd/TEMP1.CH12
- net /houskeeping/TEMP1.CH13 renamed /rtd/TEMP1.CH13
- net /houskeeping/TEMP1.CH14 renamed /rtd/TEMP1.CH14
- net /houskeeping/TEMP1.CH15 renamed /rtd/TEMP1.CH15
- net /houskeeping/TEMP1.CH16 renamed /rtd/TEMP1.CH16
- net /houskeeping/TEMP1.CH17 renamed /rtd/TEMP1.CH17
- net /houskeeping/TEMP1.CH18 renamed /rtd/TEMP1.CH18
- net /houskeeping/TEMP1.CH19 renamed /rtd/TEMP1.CH19
- net /houskeeping/TEMP1.CH20 renamed /rtd/TEMP1.CH20
- net /houskeeping/TEMP1.CH3 renamed /rtd/TEMP1.CH3
- net /houskeeping/TEMP1.CH4 renamed /rtd/TEMP1.CH4
- net /houskeeping/TEMP1.CH5 renamed /rtd/TEMP1.CH5
- net /houskeeping/TEMP1.CH6 renamed /rtd/TEMP1.CH6
- net /houskeeping/TEMP1.CH7 renamed /rtd/TEMP1.CH7
- net /houskeeping/TEMP1.CH8 renamed /rtd/TEMP1.CH8
- net /houskeeping/TEMP1.CH9 renamed /rtd/TEMP1.CH9
- net /houskeeping/TEMP1.RSENSE renamed /rtd/TEMP1.RSENSE
- net /houskeeping/TEMP1_INTRPT renamed /rtd/TEMP1_INTRPT
- net /houskeeping/TEMP1_nRESET renamed /rtd/TEMP1_nRESET
- net /houskeeping/TEMP2.CH10 renamed /rtd/TEMP2.CH10
- net /houskeeping/TEMP2.CH11 renamed /rtd/TEMP2.CH11
- net /houskeeping/TEMP2.CH12 renamed /rtd/TEMP2.CH12
- net /houskeeping/TEMP2.CH13 renamed /rtd/TEMP2.CH13
- net /houskeeping/TEMP2.CH14 renamed /rtd/TEMP2.CH14
- net /houskeeping/TEMP2.CH15 renamed /rtd/TEMP2.CH15
- net /houskeeping/TEMP2.CH16 renamed /rtd/TEMP2.CH16
- net /houskeeping/TEMP2.CH17 renamed /rtd/TEMP2.CH17
- net /houskeeping/TEMP2.CH18 renamed /rtd/TEMP2.CH18
- net /houskeeping/TEMP2.CH19 renamed /rtd/TEMP2.CH19
- net /houskeeping/TEMP2.CH20 renamed /rtd/TEMP2.CH20
- net /houskeeping/TEMP2.CH3 renamed /rtd/TEMP2.CH3
- net /houskeeping/TEMP2.CH4 renamed /rtd/TEMP2.CH4
- net /houskeeping/TEMP2.CH5 renamed /rtd/TEMP2.CH5
- net /houskeeping/TEMP2.CH6 renamed /rtd/TEMP2.CH6
- net /houskeeping/TEMP2.CH7 renamed /rtd/TEMP2.CH7
- net /houskeeping/TEMP2.CH8 renamed /rtd/TEMP2.CH8
- net /houskeeping/TEMP2.CH9 renamed /rtd/TEMP2.CH9
- net /houskeeping/TEMP2.RSENSE renamed /rtd/TEMP2.RSENSE
- net /houskeeping/TEMP2_INTRPT renamed /rtd/TEMP2_INTRPT
- net /houskeeping/TEMP2_nRESET renamed /rtd/TEMP2_nRESET
- net /houskeeping/VREF1 renamed /rtd/VREF1
- net /houskeeping/VREF2 renamed /rtd/VREF2
- net /houskeeping/VREFBYP1 renamed /rtd/VREFBYP1
- net /houskeeping/VREFBYP2 renamed /rtd/VREFBYP2
- net /microcontroller/ETH.LEDA renamed /eth_phy/ETH.LEDA
- net /microcontroller/ETH.LEDB renamed /eth_phy/ETH.LEDB
- net /microcontroller/SPI.nCS3 renamed /imu/SPI.nCS3
- net /microcontroller/SPI.nCS4 renamed /imu/SPI.nCS4
- U1 pad 1: /microcontroller/SPI.nCS2 -> /imu/SPI.nCS2
- U1 pad 2: /microcontroller/SPI.nCS1 -> /imu/SPI.nCS1
- U1 pad 34: /microcontroller/SPI.SCK -> /imu/SPI.SCK
- U1 pad 35: /microcontroller/SPI.SDI -> /imu/SPI.SDI
- U1 pad 36: /microcontroller/SPI.SDO -> /imu/SPI.SDO
- U1 pad 46: /microcontroller/ETH.RX_N -> /eth_phy/ETH.RX_N
- U1 pad 47: /microcontroller/ETH.RX_P -> /eth_phy/ETH.RX_P
- U1 pad 50: /microcontroller/ETH.TX_N -> /eth_phy/ETH.TX_N
- U1 pad 51: /microcontroller/ETH.TX_P -> /eth_phy/ETH.TX_P
- U18 pad 38: /houskeeping/SPI.SCK -> /imu/SPI.SCK
- U18 pad 39: /houskeeping/SPI.SDI -> /imu/SPI.SDI
- U18 pad 40: /houskeeping/SPI.SDO -> /imu/SPI.SDO
- U18 pad 41: /houskeeping/SPI.nCS2 -> /imu/SPI.nCS2
- U19 pad 38: /houskeeping/SPI.SCK -> /imu/SPI.SCK
- U19 pad 39: /houskeeping/SPI.SDI -> /imu/SPI.SDI
- U19 pad 40: /houskeeping/SPI.SDO -> /imu/SPI.SDO
- U19 pad 41: /houskeeping/SPI.nCS1 -> /imu/SPI.nCS1
Other:
- board outline added: 116.8 x 59.7 mm

Commit message: adding housekeeping board
Parts:
- removed D4: R, Capacitor_SMD:C_0402_1005Metric
- added C38: 0.1µF, Capacitor_SMD:C_0603_1608Metric, F.Cu at (101.6, 62.2)
- added C39: 0.1µF, Capacitor_SMD:C_0603_1608Metric, F.Cu at (101.6, 67.3)
- added C40: 0.1µF, Capacitor_SMD:C_0603_1608Metric, F.Cu at (101.6, 72.4)
- added C41: 0.1µF, Capacitor_SMD:C_0603_1608Metric, F.Cu at (107.2, 62.2)
- added C42: 0.1µF, Capacitor_SMD:C_0603_1608Metric, F.Cu at (107.2, 67.3)
- added C43: 0.1µF, Capacitor_SMD:C_0603_1608Metric, F.Cu at (107.2, 72.4)
- added C44: 0.1µF, Capacitor_SMD:C_0603_1608Metric, F.Cu at (170.2, 79.9)
- added C45: 0.1µF, Capacitor_SMD:C_0603_1608Metric, F.Cu at (172.6, 77.3)
- added C46: 0.1µF, Capacitor_SMD:C_0603_1608Metric, F.Cu at (172.3, 81.9)
- added C47: 0.1µF, Capacitor_SMD:C_0603_1608Metric, F.Cu at (172.3, 85.0)
- added C49: 0.1µF, Capacitor_SMD:C_1206_3216Metric, B.Cu at (105.2, 81.3)
- added C50: 0.1µF, Capacitor_SMD:C_1206_3216Metric, B.Cu at (114.4, 84.1)
- added C51: 0.1µF, Capacitor_SMD:C_1206_3216Metric, B.Cu at (117.4, 86.3)
- added C52: 56pF 5%, Capacitor_SMD:C_0603_1608Metric, F.Cu at (117.9, 87.4)
- added C53: 56pF 5%, Capacitor_SMD:C_0603_1608Metric, F.Cu at (116.6, 85.2)
- added C54: 10µF, 16V, Capacitor_SMD:C_0603_1608Metric, B.Cu at (134.1, 65.0)
- added C55: 0.1µF, Capacitor_SMD:C_0603_1608Metric, F.Cu at (113.2, 72.3)
- added C56: 0.1µF, Capacitor_SMD:C_0603_1608Metric, F.Cu at (113.9, 66.3)
- added FID1: Fiducial, Fiducial:Fiducial_1mm_Mask2mm, F.Cu at (112.4, 57.7)
- added FID2: Fiducial, Fiducial:Fiducial_1mm_Mask2mm, F.Cu at (174.0, 103.9)
- added G***: LOGO, LOGO, F.Cu at (183.4, 88.1)
- added J2: Conn_02x08_Odd_Even, Connector_PinHeader_2.54mm:PinHeader_2x08_P2.54mm_Vertical, B.Cu at (93.5, 58.2)
- added J7: Conn_01x16, Connector_PinHeader_2.54mm:PinHeader_1x16_P2.54mm_Vertical, F.Cu at (182.1, 51.1)
- added J9: Conn_01x03, Connector_PinSocket_2.54mm:PinSocket_1x03_P2.54mm_Vertical, F.Cu at (128.8, 51.1)
- added R25: 4.7kΩ, Resistor_SMD:R_0603_1608Metric, B.Cu at (153.2, 57.1)
- added R26: 4.7kΩ, Resistor_SMD:R_0603_1608Metric, B.Cu at (151.6, 57.1)
- added R27: 4.7kΩ, Resistor_SMD:R_0603_1608Metric, F.Cu at (106.4, 59.7)
- added R28: 4.7kΩ, Resistor_SMD:R_0603_1608Metric, F.Cu at (106.4, 64.8)
- added R29: 4.7kΩ, Resistor_SMD:R_0603_1608Metric, F.Cu at (106.4, 69.8)
- added SW1: SW_Push_LED_Wuerth_WS-TASL, Button_Switch_SMD:SW_Tactile_SPST_Wuerth_WS-TASL, F.Cu at (110.0, 51.8)
- added SW2: SW_Push_LED_Wuerth_WS-TASL, Button_Switch_SMD:SW_Tactile_SPST_Wuerth_WS-TASL, F.Cu at (120.1, 51.8)
- added TP1: TestPoint, TestPoint:TestPoint_Loop_D2.60mm_Drill1.4mm_Beaded, F.Cu at (138.9, 51.1)
- added TP10: TestPoint, TestPoint:TestPoint_THTPad_D2.0mm_Drill1.0mm, F.Cu at (166.1, 81.9)
- added TP11: TestPoint, TestPoint:TestPoint_THTPad_D2.0mm_Drill1.0mm, F.Cu at (157.6, 73.4)
- added TP12: TestPoint, TestPoint:TestPoint_THTPad_D2.0mm_Drill1.0mm, F.Cu at (141.2, 79.6)
- added TP13: TestPoint, TestPoint:TestPoint_THTPad_D2.0mm_Drill1.0mm, F.Cu at (141.2, 84.5)
- added TP14: TestPoint, TestPoint:TestPoint_THTPad_D2.0mm_Drill1.0mm, F.Cu at (151.5, 73.4)
- added TP16: TestPoint, TestPoint:TestPoint_THTPad_D2.0mm_Drill1.0mm, F.Cu at (122.7, 88.9)
- added TP2: TestPoint, TestPoint:TestPoint_THTPad_D2.0mm_Drill1.0mm, F.Cu at (144.8, 88.9)
- added TP3: TestPoint, TestPoint:TestPoint_Pad_1.5x1.5mm, F.Cu at (138.7, 62.1)
- added TP4: TestPoint, TestPoint:TestPoint_THTPad_D2.0mm_Drill1.0mm, F.Cu at (154.6, 73.4)
- added TP5: TestPoint, TestPoint:TestPoint_THTPad_D2.0mm_Drill1.0mm, F.Cu at (164.5, 71.6)
- added TP6: TestPoint, TestPoint:TestPoint_THTPad_D2.0mm_Drill1.0mm, F.Cu at (164.5, 68.6)
- added TP7: TestPoint, TestPoint:TestPoint_THTPad_D2.0mm_Drill1.0mm, F.Cu at (164.5, 65.5)
- added TP8: TestPoint, TestPoint:TestPoint_THTPad_D2.0mm_Drill1.0mm, F.Cu at (161.4, 65.5)
- added TP9: TestPoint, TestPoint:TestPoint_THTPad_D2.0mm_Drill1.0mm, F.Cu at (166.1, 78.9)
- added U2: 74LVC1G86, Package_TO_SOT_SMD:SOT-23-5, F.Cu at (168.4, 63.5)
- added U5: 74LVC1G08, Package_TO_SOT_SMD:SOT-23-5, F.Cu at (173.0, 70.6)
- added Y1: 25 MHz, Crystal:Crystal_SMD_3225-4Pin_3.2x2.5mm, F.Cu at (120.7, 65.3)
- C1, C12, C17, C18, C22, C23, C34, C35: footprint Capacitor_SMD:C_0402_1005Metric -> Capacitor_SMD:C_0603_1608Metric
- C10, C11, C36, C37, C5, C6, C7, C8, C9: footprint Capacitor_SMD:C_0402_1005Metric -> Capacitor_SMD:C_0603_1608Metric; moved to B.Cu
- C13, C14, C24, C25: value 22µF -> 0.1µF; footprint Capacitor_SMD:C_1206_3216Metric -> Capacitor_SMD:C_0603_1608Metric
- C15, C19: footprint Capacitor_SMD:C_0805_2012Metric -> Capacitor_SMD:C_1206_3216Metric
- C16, C20: value 10µF -> 0.1µF; footprint Capacitor_SMD:C_0805_2012Metric -> Capacitor_SMD:C_0603_1608Metric
- C2, C3: value 33pF 5% -> 10pF 1%
- C21: value 1µF -> 0.1µF
- C28, C29, C30, C31, C32, C33, C4: moved to B.Cu
- H1, H2, H3, H4: footprint MountingHole:MountingHole_3.2mm_M3_Pad -> MountingHole:MountingHole_0.112in_Pad
- J4: value Conn_02x10_Row_Letter_First -> Conn_02x06_Row_Letter_First; footprint Connector_Harwin:Harwin_JTek-Male_2x10_P2.00mm_Horizontal -> Connector_Harwin:Harwin_JTek-Male_2x6_P2.00mm_Horizontal
- L1, L3: value 4.7 µH -> 120Ω; footprint Inductor_SMD:L_Wuerth_MAPI-4030 -> Resistor_SMD:R_0603_1608Metric
- R10: value 50kΩ 1% -> 180Ω
- R11: value 22kΩ 1% -> 47Ω; footprint Resistor_SMD:R_0603_1608Metric -> Resistor_SMD:R_1210_3225Metric; moved to B.Cu
- R12, R13: value 500Ω -> 49.9Ω 1%
- R14, R19, R20, R21, R22: value 500Ω -> 4.7kΩ
- R16, R17: value 4.7kΩ -> 75Ω
- R23, R24: value 150Ω -> 4.7kΩ
- R3: value 4.7kΩ -> 150Ω
- R5: value 12.6kΩ 1% -> 4.7kΩ
- R6: value 22kΩ 1% -> 180Ω
- R7: value 180 kΩ -> 200Ω
- R8, R9: value 180 kΩ -> 49.9Ω 1%; moved to B.Cu
- U10, U6, U7, U9: moved to F.Cu
- U12, U13, U14: value NBA3N011S -> SN74LVC1T45DBV; footprint Package_TO_SOT_SMD:SOT-23-5 -> Package_TO_SOT_SMD:SOT-23-6
- U15: value NBA3N011S -> BME680; footprint Package_TO_SOT_SMD:SOT-23-5 -> Package_LGA:Bosch_LGA-8_3x3mm_P0.8mm_ClockwisePinNumbering
- U17: value TPS54294 -> TXB0108DQSR; footprint Package_DFN_QFN:Texas_S-PVQFN-N16_EP2.7x2.7mm -> Package_SON:USON-20_2x4mm_P0.4mm
- moved J4 212.1 mm to (191.8, 69.6)
- moved J5 211.4 mm to (97.8, 92.8)
- moved H1 208.8 mm to (199.4, 51.8)
- moved H2 208.8 mm to (90.2, 51.8)
- moved H3 208.8 mm to (183.5, 103.9)
- moved H4 208.8 mm to (111.1, 103.9)
- moved J3 208.4 mm to (144.8, 96.9)
- moved C13 93.3 mm to (184.4, 66.8)
- moved U20 89.2 mm to (170.1, 83.8), turned to 90 degrees
- moved C14 81.9 mm to (179.1, 69.6)
- moved C20 78.4 mm to (173.0, 68.1), turned to 180 degrees
- moved C1 76.7 mm to (147.6, 64.0), turned to 180 degrees
- moved C22 69.3 mm to (172.0, 66.0)
- moved C18 69.2 mm to (184.4, 78.0)
- moved C16 69.1 mm to (184.4, 72.4)
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- renumbered RSENSE2 to RSENSE1, RSENSE1 to RSENSE2
Connections:
- C11 pad 2: /microcontroller/AVSS -> GND
- C12 pad 1: unconnected-(C12-Pad1) -> +3V3
- C12 pad 2: unconnected-(C12-Pad2) -> GND
- C13 pad 1: GND -> +3V3
- C13 pad 2: +1V2 -> GND
- C14 pad 1: GND -> +3V3
- C14 pad 2: +1V2 -> GND
- C16 pad 1: GND -> +3V3
- C16 pad 2: +5V -> GND
- C17 pad 1: Net-(C17-Pad1) -> +3V3
- C17 pad 2: Net-(C17-Pad2) -> GND
- C18 pad 1: GND -> +3V3
- C18 pad 2: +5V -> GND
- C20 pad 1: GND -> +3V3
- C20 pad 2: +5V -> GND
- C21 pad 1: Net-(C21-Pad1) -> +3V3
- C22 pad 1: Net-(C22-Pad1) -> +3V3
- C22 pad 2: Net-(C22-Pad2) -> GND
- C23 pad 1: GND -> +3V3
- C23 pad 2: +5V -> GND
- C24 pad 2: +2V5 -> +5V
- C25 pad 2: +2V5 -> +3V3
- H1 pad 1: unconnected-(H1-Pad1) -> GNDPWR
- H2 pad 1: unconnected-(H2-Pad1) -> GNDPWR
- H3 pad 1: unconnected-(H3-Pad1) -> GNDPWR
- H4 pad 1: unconnected-(H4-Pad1) -> GNDPWR
- J3 pad a1: /rtd_header/TEMP1.RSENSE -> /rtd/TEMP1.RSENSE
- J3 pad a12: /rtd_header/TEMP2.RSENSE -> /rtd/TEMP2.RSENSE
- J3 pad a13: /rtd_header/TEMP2.RSENSE -> /rtd/TEMP2.RSENSE
- J3 pad a14: /rtd_header/TEMP2.RSENSE -> /rtd/TEMP2.RSENSE
- J3 pad a15: /rtd_header/TEMP2.RSENSE -> /rtd/TEMP2.RSENSE
- J3 pad a16: /rtd_header/TEMP2.RSENSE -> /rtd/TEMP2.RSENSE
- J3 pad a17: /rtd_header/TEMP2.RSENSE -> /rtd/TEMP2.RSENSE
- J3 pad a18: /rtd_header/TEMP2.RSENSE -> /rtd/TEMP2.RSENSE
- J3 pad a19: /rtd_header/TEMP2.RSENSE -> /rtd/TEMP2.RSENSE
- J3 pad a2: /rtd_header/TEMP1.RSENSE -> /rtd/TEMP1.RSENSE
- J3 pad a20: /rtd_header/TEMP2.RSENSE -> /rtd/TEMP2.RSENSE
- J3 pad a3: /rtd_header/TEMP1.RSENSE -> /rtd/TEMP1.RSENSE
- J3 pad a4: /rtd_header/TEMP1.RSENSE -> /rtd/TEMP1.RSENSE
- J3 pad a5: /rtd_header/TEMP1.RSENSE -> /rtd/TEMP1.RSENSE
- J3 pad a6: /rtd_header/TEMP1.RSENSE -> /rtd/TEMP1.RSENSE
- J3 pad a7: /rtd_header/TEMP1.RSENSE -> /rtd/TEMP1.RSENSE
- J3 pad a8: /rtd_header/TEMP1.RSENSE -> /rtd/TEMP1.RSENSE
- J3 pad a9: /rtd_header/TEMP1.RSENSE -> /rtd/TEMP1.RSENSE
- J3 pad b1: /rtd_header/TEMP1.CH3 -> /rtd/TEMP1.CH20
- J3 pad b12: /rtd_header/TEMP2.CH3 -> /rtd/TEMP2.CH20
- J3 pad b13: /rtd_header/TEMP2.CH5 -> /rtd/TEMP2.CH18
- J3 pad b14: /rtd_header/TEMP2.CH7 -> /rtd/TEMP2.CH16
- J3 pad b15: /rtd_header/TEMP2.CH9 -> /rtd/TEMP2.CH14
- J3 pad b16: /rtd_header/TEMP2.CH11 -> /rtd/TEMP2.CH12
- J3 pad b17: /rtd_header/TEMP2.CH13 -> /rtd/TEMP2.CH10
- J3 pad b18: /rtd_header/TEMP2.CH15 -> /rtd/TEMP2.CH8
- J3 pad b19: /rtd_header/TEMP2.CH17 -> /rtd/TEMP2.CH6
- J3 pad b2: /rtd_header/TEMP1.CH5 -> /rtd/TEMP1.CH18
- J3 pad b20: /rtd_header/TEMP2.CH19 -> /rtd/TEMP2.CH4
- J3 pad b3: /rtd_header/TEMP1.CH7 -> /rtd/TEMP1.CH16
- J3 pad b4: /rtd_header/TEMP1.CH9 -> /rtd/TEMP1.CH14
- J3 pad b5: /rtd_header/TEMP1.CH11 -> /rtd/TEMP1.CH12
- J3 pad b6: /rtd_header/TEMP1.CH13 -> /rtd/TEMP1.CH10
- J3 pad b7: /rtd_header/TEMP1.CH15 -> /rtd/TEMP1.CH8
- J3 pad b8: /rtd_header/TEMP1.CH17 -> /rtd/TEMP1.CH6
- J3 pad b9: /rtd_header/TEMP1.CH19 -> /rtd/TEMP1.CH4
- J3 pad c1: /rtd_header/TEMP1.CH4 -> /rtd/TEMP1.CH19
- J3 pad c12: /rtd_header/TEMP2.CH4 -> /rtd/TEMP2.CH19
- J3 pad c13: /rtd_header/TEMP2.CH6 -> /rtd/TEMP2.CH17
- J3 pad c14: /rtd_header/TEMP2.CH8 -> /rtd/TEMP2.CH15
- J3 pad c15: /rtd_header/TEMP2.CH10 -> /rtd/TEMP2.CH13
- J3 pad c16: /rtd_header/TEMP2.CH12 -> /rtd/TEMP2.CH11
- J3 pad c17: /rtd_header/TEMP2.CH14 -> /rtd/TEMP2.CH9
- J3 pad c18: /rtd_header/TEMP2.CH16 -> /rtd/TEMP2.CH7
- J3 pad c19: /rtd_header/TEMP2.CH18 -> /rtd/TEMP2.CH5
- J3 pad c2: /rtd_header/TEMP1.CH6 -> /rtd/TEMP1.CH17
- J3 pad c20: /rtd_header/TEMP2.CH20 -> /rtd/TEMP2.CH3
- J3 pad c3: /rtd_header/TEMP1.CH8 -> /rtd/TEMP1.CH15
- J3 pad c4: /rtd_header/TEMP1.CH10 -> /rtd/TEMP1.CH13
- J3 pad c5: /rtd_header/TEMP1.CH12 -> /rtd/TEMP1.CH11
- J3 pad c6: /rtd_header/TEMP1.CH14 -> /rtd/TEMP1.CH9
- J3 pad c7: /rtd_header/TEMP1.CH16 -> /rtd/TEMP1.CH7
- J3 pad c8: /rtd_header/TEMP1.CH18 -> /rtd/TEMP1.CH5
- J3 pad c9: /rtd_header/TEMP1.CH20 -> /rtd/TEMP1.CH3
- J4 pad a1: /sync/SYNC1- -> /sync/SYNC1+
- J4 pad a2: /sync/SYNC1+ -> /sync/SYNC1-
- J4 pad a3: unconnected-(J4-Pada3) -> /sync/SYNC3+
- J4 pad a4: unconnected-(J4-Pada4) -> /sync/SYNC3-
- J4 pad a5: unconnected-(J4-Pada5) -> /sync/SYNC5+
- J4 pad a6: unconnected-(J4-Pada6) -> /sync/SYNC5-
- J4 pad b1: /sync/SYNC2- -> /sync/SYNC2+
- J4 pad b2: /sync/SYNC2+ -> /sync/SYNC2-
- J4 pad b3: unconnected-(J4-Padb3) -> /sync/SYNC4+
- J4 pad b4: unconnected-(J4-Padb4) -> /sync/SYNC4-
- J4 pad b5: unconnected-(J4-Padb5) -> /sync/SYNC6+
- J4 pad b6: unconnected-(J4-Padb6) -> /sync/SYNC6-
- J5 pad 1: unconnected-(J5-Pad1) -> Net-(J5-LED1+)
- J5 pad 10: unconnected-(J5-Pad10) -> Net-(J5-VC1_N)
- J5 pad 11: unconnected-(J5-Pad11) -> Net-(J5-VC2_N)
- J5 pad 12: unconnected-(J5-Pad12) -> Net-(J5-VC2_N)
- J5 pad 13: unconnected-(J5-Pad13) -> Net-(J5-LED2+)
- J5 pad 14: unconnected-(J5-Pad14) -> GND
- J5 pad 2: unconnected-(J5-Pad2) -> GND
- J5 pad 3: /eth_phy/ETH.TX_P -> /eth_phy/ETHTXJ_P
- J5 pad 4: /eth_phy/ETH.TX_N -> /eth_phy/ETHTXJ_N
- J5 pad 5: unconnected-(J5-Pad5) -> +3V3
- J5 pad 9: unconnected-(J5-Pad9) -> Net-(J5-VC1_N)
- J5 pad EP1: unconnected-(J5-PadEP1) -> GNDPWR
- J5 pad EP2: unconnected-(J5-PadEP2) -> GNDPWR
- L1 pad 1: +1V2 -> /eth_phy/ETH.TX_P
- L1 pad 2: Net-(C17-Pad2) -> /eth_phy/ETHTXJ_P
- L3 pad 1: Net-(C22-Pad1) -> /eth_phy/ETH.TX_N
- L3 pad 2: +2V5 -> /eth_phy/ETHTXJ_N
- R10 pad 1: +2V5 -> Net-(J5-LED2+)
- R10 pad 2: Net-(R10-Pad2) -> /eth_phy/ETH.LEDB
- R11 pad 1: Net-(R10-Pad2) -> GNDPWR
- R12 pad 1: +3V3 -> Net-(C50-Pad1)
- R12 pad 2: Net-(D1-Pad2) -> /eth_phy/ETH.RX_P
- R13 pad 1: /power/3V3_SNOOZE -> /eth_phy/ETH.RX_N
- R13 pad 2: Net-(D2-Pad2) -> Net-(C50-Pad1)
- R14 pad 1: /power/3V3_EN -> GND
- R14 pad 2: Net-(D3-Pad2) -> /microcontroller/SPI.SDI
- R15 pad 1: +5V -> GND
- R15 pad 2: /power/1V2_PG -> /microcontroller/SPI.SCK
- R16 pad 1: +5V -> Net-(C49-Pad1)
- R16 pad 2: /power/2V5_PG -> Net-(J5-VC1_N)
- R17 pad 1: +5V -> Net-(C49-Pad1)
- R17 pad 2: /power/1V2_EN -> Net-(J5-VC2_N)
- R18 pad 1: +5V -> GND
- R18 pad 2: /power/2V5_EN -> /microcontroller/SPI.SDO
- R19 pad 1: +5V -> /microcontroller/SPI.nCS1
- R19 pad 2: Net-(D4-Pad2) -> +3V3
- R20 pad 1: /power/1V2_EN -> /microcontroller/SPI.nCS2
- R20 pad 2: Net-(D5-Pad2) -> +3V3
- R21 pad 1: +5V -> /microcontroller/SPI.nCS3
- R21 pad 2: Net-(D6-Pad2) -> +3V3
- R22 pad 1: /power/2V5_EN -> /microcontroller/SPI.nCS4
- R22 pad 2: Net-(D7-Pad2) -> +3V3
- R23 pad 1: Net-(D8-Pad2) -> /microcontroller/SPI.nCS6
- R23 pad 2: /eth_phy/LEDA -> +3V3
- R24 pad 1: Net-(D9-Pad2) -> /microcontroller/SPI.nCS5
- R24 pad 2: /eth_phy/LEDB -> +3V3
- R5 pad 1: Net-(R5-Pad1) -> /microcontroller/TEMP_nRESET
- R5 pad 2: +1V2 -> +3V3
- R6 pad 1: GND -> Net-(J5-LED1+)
- R6 pad 2: Net-(R5-Pad1) -> /eth_phy/ETH.LEDA
- R7 pad 2: +3V3 -> +5V
- R8 pad 1: /power/3V3_PG -> +3V3
- R8 pad 2: +3V3 -> /eth_phy/ETHTXJ_P
- R9 pad 1: /power/3V3_SNOOZE -> /eth_phy/ETHTXJ_N
- R9 pad 2: GND -> +3V3
- U1 pad 1: /imu/SPI.nCS2 -> /microcontroller/SPI.nCS2
- U1 pad 10: +2V5 -> /microcontroller/VDDCORE
- U1 pad 18: GND -> +3V3
- U1 pad 2: /imu/SPI.nCS1 -> /microcontroller/SPI.nCS1
- U1 pad 20: /microcontroller/AVSS -> GND
- U1 pad 21: unconnected-(U1-Pad21) -> /microcontroller/RA3
- U1 pad 22: unconnected-(U1-Pad22) -> /microcontroller/RA2
- U1 pad 27: unconnected-(U1-Pad27) -> /microcontroller/RA5
- U1 pad 28: unconnected-(U1-Pad28) -> /microcontroller/RA4
- U1 pad 29: /microcontroller/2V5_EN -> /microcontroller/RC1
- U1 pad 30: /microcontroller/1V2_EN -> /microcontroller/RC0
- U1 pad 33: /microcontroller/3V3_SNOOZE -> /microcontroller/RC2
- U1 pad 34: /imu/SPI.SCK -> /microcontroller/SPI.SCK
- U1 pad 35: /imu/SPI.SDI -> /microcontroller/SPI.SDI
- U1 pad 36: /imu/SPI.SDO -> /microcontroller/SPI.SDO
- U1 pad 43: /microcontroller/2V5_PG -> unconnected-(U1-KBI1/RB5-Pad43)
- U1 pad 44: /microcontroller/1V2_PG -> unconnected-(U1-KBI0/RB4-Pad44)
- U1 pad 58: unconnected-(U1-Pad58) -> /microcontroller/TEMP2_READY
- U1 pad 59: unconnected-(U1-Pad59) -> /microcontroller/TEMP_nRESET
- U1 pad 60: unconnected-(U1-Pad60) -> /microcontroller/TEMP1_READY
- U1 pad 61: /microcontroller/TEMP2_READY -> /microcontroller/SPI.nCS6
- U1 pad 62: /microcontroller/TEMP1_READY -> /microcontroller/SPI.nCS5
- U1 pad 63: /imu/SPI.nCS4 -> /microcontroller/SPI.nCS4
- U1 pad 64: /imu/SPI.nCS3 -> /microcontroller/SPI.nCS3
- U12 pad 3: /sync/SYNC7- -> /power/PPS
- U12 pad 4: /sync/SYNC7+ -> /power/PPS_in
- U12 pad 5: /microcontroller/INTRPT0 -> GND
- U13 pad 3: /sync/SYNC8- -> /microcontroller/INTRPT2
- U13 pad 4: /sync/SYNC8+ -> /power/SHUTTER_in
- U13 pad 5: /microcontroller/INTRPT0 -> GND
- U14 pad 3: /sync/SYNC9- -> /microcontroller/INTRPT1
- U14 pad 4: /sync/SYNC9+ -> /power/PRELAUNCH_in
- U14 pad 5: /microcontroller/INTRPT0 -> GND
- U15 pad 1: +3V3 -> GND
- U15 pad 2: GND -> /microcontroller/SPI.nCS5
- U15 pad 3: /sync/SYNC10- -> /microcontroller/SPI.SDI
- U15 pad 4: /sync/SYNC10+ -> /microcontroller/SPI.SCK
- U15 pad 5: /microcontroller/INTRPT0 -> /microcontroller/SPI.SDO
- U16 pad 3: /power/3V3_SNOOZE -> GND
- U17 pad 1: Net-(C22-Pad2) -> /power/SCK
- U17 pad 10: GND -> /power/nCS4
- U17 pad 11: Net-(C21-Pad1) -> /microcontroller/SPI.nCS4
- U17 pad 12: Net-(R10-Pad2) -> /microcontroller/SPI.nCS3
- U17 pad 13: /power/2V5_PG -> unconnected-(U17-B6-Pad13)
- U17 pad 14: /power/2V5_EN -> unconnected-(U17-B5-Pad14)
- U17 pad 16: Net-(C22-Pad1) -> +3V3
- U17 pad 17: GND -> unconnected-(U17-B4-Pad17)
- U17 pad 2: +5V -> /power/SDI
- U17 pad 3: +5V -> /power/SDO
- U17 pad 4: Net-(C17-Pad1) -> unconnected-(U17-A4-Pad4)
- U17 pad 5: Net-(C17-Pad2) -> +3V3
- U17 pad 6: GND -> +3V3
- U17 pad 7: /power/1V2_EN -> unconnected-(U17-A5-Pad7)
- U17 pad 8: /power/1V2_PG -> unconnected-(U17-A6-Pad8)
- U17 pad 9: Net-(R5-Pad1) -> /power/nCS3
- U18 pad 37: /rtd/TEMP2_INTRPT -> /microcontroller/TEMP2_READY
- U18 pad 38: /imu/SPI.SCK -> /microcontroller/SPI.SCK
- U18 pad 39: /imu/SPI.SDI -> /microcontroller/SPI.SDI
- U18 pad 40: /imu/SPI.SDO -> /microcontroller/SPI.SDO
- U18 pad 41: /imu/SPI.nCS2 -> /microcontroller/SPI.nCS2
- U18 pad 42: /rtd/TEMP2_nRESET -> /microcontroller/TEMP_nRESET
- U19 pad 37: /rtd/TEMP1_INTRPT -> /microcontroller/TEMP1_READY
- U19 pad 38: /imu/SPI.SCK -> /microcontroller/SPI.SCK
- U19 pad 39: /imu/SPI.SDI -> /microcontroller/SPI.SDI
- U19 pad 40: /imu/SPI.SDO -> /microcontroller/SPI.SDO
- U19 pad 41: /imu/SPI.nCS1 -> /microcontroller/SPI.nCS1
- U19 pad 42: /rtd/TEMP1_nRESET -> /microcontroller/TEMP_nRESET
- U20 pad 1: unconnected-(U20-Pad1) -> /microcontroller/SPI.SDO
- U20 pad 12: unconnected-(U20-Pad12) -> /microcontroller/SPI.nCS6
- U20 pad 13: unconnected-(U20-Pad13) -> /microcontroller/SPI.SCK
- U20 pad 14: unconnected-(U20-Pad14) -> /microcontroller/SPI.SDI
- U20 pad 5: Net-(U20-Pad5) -> +3V3
- U20 pad 6: Net-(U20-Pad6) -> GND
- U20 pad 7: Net-(U20-Pad6) -> GND
- U20 pad 8: Net-(U20-Pad5) -> +3V3
- U3 pad 1: Net-(U2-Pad4) -> /sync/R
Routing:
- net /microcontroller/SPI.SCK: track 0.00 -> 125.4 mm, vias 0 -> 7
- net /microcontroller/SPI.SDO: track 0.00 -> 124.1 mm, vias 0 -> 6
- net /microcontroller/SPI.SDI: track 0.00 -> 122.0 mm, vias 0 -> 7
- net /microcontroller/INTRPT1: track 0.00 -> 100.1 mm, vias 0 -> 4
- net /microcontroller/INTRPT0: track 0.00 -> 93.9 mm, vias 0 -> 7
- net /power/PPS: track 0.00 -> 78.2 mm, vias 0 -> 3
- net /microcontroller/nMCLR: track 0.00 -> 75.4 mm, vias 0 -> 3
- net /microcontroller/UNLAUNCH: track 0.00 -> 61.5 mm, vias 0 -> 3
- net /microcontroller/PGD: track 0.00 -> 61.1 mm, vias 0 -> 2
- net /microcontroller/PGC: track 0.00 -> 60.7 mm, vias 0 -> 1
- net /microcontroller/INTRPT2: track 0.00 -> 59.8 mm, vias 0 -> 2
- net /microcontroller/SPI.nCS1: track 0.00 -> 53.3 mm, vias 0 -> 2
- net +5V: track 0.00 -> 51.7 mm, vias 0 -> 1
- net /eth_phy/ETH.LEDA: track 0.00 -> 51.7 mm, vias 0 -> 2
- net /microcontroller/INTRPT3: track 0.00 -> 50.0 mm
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- added copper zone on B.Cu, net +3V3
- added copper zone on F.Cu, net +3V3
- added copper zone on In2.Cu, net +3V3
- added copper zone on F.Cu, net +5V
- added copper zone on F.Cu, net /microcontroller/INTRPT1
- added copper zone on F.Cu, net /microcontroller/INTRPT2
- added copper zone on F.Cu, net /microcontroller/UNLAUNCH
- added copper zone on F.Cu, net /power/3V3_EN
- added copper zone on F.Cu, net /power/PPS
- added copper zone on B.Cu, net /rtd/TEMP1.RSENSE
- added copper zone on B.Cu, net /rtd/TEMP2.RSENSE
- added copper zone on B.Cu, net /rtd/VREF1
- added copper zone on F.Cu, net /rtd/VREF1
- added copper zone on B.Cu, net /rtd/VREF2
- added copper zone on F.Cu, net /rtd/VREF2
- added copper zone on B.Cu, net GND
- added copper zone on F.Cu, net GND
- added copper zone on In1.Cu, net GND
- added copper zone on In2.Cu, net GND
- added copper zone on B.Cu, net GNDPWR
- added copper zone on F.Cu, net GNDPWR
- added copper zone on In1.Cu, net GNDPWR
- added copper zone on In2.Cu, net GNDPWR
- added copper zone on B.Cu, net Net-(C50-Pad1)
- added copper zone on F.Cu, net Net-(U16-SW)
Other:
- outline, holes or cut-outs redrawn
- copper layers 2 -> 4
- board text added: "0"
- board text added: "0 mils"
- board text added: "0.021"
- board text added: "0.022"
- board text added: "0.033"
- board text added: "0.6 mils"
- board text added: "1"
- board text added: "1.2 mils"
- board text added: "1.8 mils"
- board text added: "2.7"
- board text added: "3.99"
- board text added: "39 mils"
- board text added: "4.71"
- board text added: "7.64 mils"
- board text added: "B.Cu"
- board text added: "B.Mask"
- board text added: "B.Paste"
- board text added: "B.Silkscreen"
- board text added: "Bottom Silk Screen"
- board text added: "Bottom Solder Mask"
- board text added: "Bottom Solder Paste"
- board text added: "Color"
- board text added: "Dielectric 1"
- board text added: "Dielectric 2"
- board text added: "Dielectric 3"
- board text added: "Epsilon R"
- board text added: "F.Cu"
- board text added: "F.Mask"
- board text added: "F.Paste"
- board text added: "F.Silkscreen"
- board text added: "FR4"
- board text added: "Green"
- board text added: "In1.Cu"
- board text added: "In2.Cu"
- board text added: "Layer Name"
- board text added: "Loss Tangent"
- board text added: "Mar 2023"
- board text added: "Material"
- board text added: "Not specified"
- board text added: "Taiyo-SM"
- board text added: "Thickness (mils)"
- board text added: "Top Silk Screen"
- board text added: "Top Solder Mask"
- board text added: "Top Solder Paste"
- board text added: "Type"
- board text added: "White"
- board text added: "copper"
- board text added: "core"
- board text added: "formatter/hk"
- board text added: "prepreg"
- board text added: "v1"
