File: plenum/rtd.kicad_sch (KiCad schematic)
At the start: 16 parts, among them U18 LTC2983, U19 LTC2983

Commit message: adding housekeeping board
Parts:
- added TP10 (x4): TestPoint, TestPoint:TestPoint_THTPad_D2.0mm_Drill1.0mm, symbol Connector:TestPoint
- C34, C35, C36, C37: footprint Capacitor_SMD:C_0402_1005Metric -> Capacitor_SMD:C_0603_1608Metric
- renumbered RSENSE2 to RSENSE1, RSENSE1 to RSENSE2
Connections:
- net TEMP1_INTRPT: now also TP10.1
- net TEMP2_INTRPT: now also TP10.1
- net at RSENSE2.1, U18.16 (CH1): now also TP10.1
- net at RSENSE1.1, U19.16 (CH1): now also TP10.1
