File: plenum/sync.kicad_sch (KiCad schematic)
At the start: 16 parts, among them J4 Conn_02x10_Row_Letter_First, U10 NBA3N011S, U11 NBA3N011S, U12 NBA3N011S, U13 NBA3N011S, U14 NBA3N011S, U15 NBA3N011S, U2 74LVC1G86, U3 74LVC1G02, U4 74LVC1G02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

Commit message: adding housekeeping board
Parts:
- removed J4: Conn_02x10_Row_Letter_First, Connector_Harwin:Harwin_JTek-Male_2x10_P2.00mm_Horizontal, symbol Connector_Generic:Conn_02x10_Row_Letter_First
- removed U12, U13, U14, U15: NBA3N011S, Package_TO_SOT_SMD:SOT-23-5, symbol Interface_LineDriver:NBA3N011S
- added C13, C14, C16, C17, C18, C20, C21, C22, C23: 0.1µF, Capacitor_SMD:C_0603_1608Metric, symbol Device:C
- added J4: Conn_02x06_Row_Letter_First, Connector_Harwin:Harwin_JTek-Male_2x6_P2.00mm_Horizontal, symbol Connector_Generic_MountingPin:Conn_02x06_Row_Letter_First_MountingPin
- added TP1 (x4): TestPoint, TestPoint:TestPoint_THTPad_D2.0mm_Drill1.0mm, symbol Connector:TestPoint
- C12: footprint Capacitor_SMD:C_0402_1005Metric -> Capacitor_SMD:C_0603_1608Metric
- U2, U5: footprint (none) -> Package_TO_SOT_SMD:SOT-23-5
Connections:
- net +3V3: now also C12.1, C13.1, C14.1, C16.1, C17.1, C18.1, C20.1, C21.1, C22.1, C23.1
- net GND: now also C12.2, C13.2, C14.2, C16.2, C17.2, C18.2, C20.2, C21.2, C22.2, C23.2
- net PPS: now also TP1.1
- net Q: now also TP1.1
- net SYNC: now also TP1.1
- net SYNC1+: now also J4.a1 (Pin_a1)
- net SYNC1-: now also J4.a2 (Pin_a2)
- net SYNC2+: now also J4.b1 (Pin_b1)
- net SYNC2-: now also J4.b2 (Pin_b2)
- net SYNC3+: now also J4.a3 (Pin_a3)
- net SYNC3-: now also J4.a4 (Pin_a4)
- net SYNC4+: now also J4.b3 (Pin_b3)
- net SYNC4-: now also J4.b4 (Pin_b4)
- net SYNC5+: now also J4.a5 (Pin_a5)
- net SYNC5-: now also J4.a6 (Pin_a6)
- net SYNC6+: now also J4.b5 (Pin_b5)
- net SYNC6-: now also J4.b6 (Pin_b6)
- net nQ: now also TP1.1
- net R: now reaches U2.4, U3.1
- net LAUNCH renamed PRELAUNCH
- new net GNDPWR: J4.MP (MountPin)
Other:
- note added: "Something like Harwin M80-5401242 (2x6 pins)"
- moved on the sheet: C12
